File: cad/prs_leaf_board/prs_leaf_board.kicad_pcb (KiCad board)
At the start: 2 copper layers, 152.4 x 76.2 mm, 11 parts, among them J101 Conn_01x07

Commit message: rev1
Parts:
- added H101: MountingHole_Pad, MountingHole:MountingHole_6.4mm_M6_Pad_Via, F.Cu at (79.6, 73.6)
- added H102: MountingHole_Pad, MountingHole:MountingHole_6.4mm_M6_Pad_Via, F.Cu at (79.6, 103.6)
- moved J101 12.4 mm to (84.0, 44.0)
- renumbered H101 to H103, H102 to H104, H103 to H105, H104 to H106, H105 to H107, H106 to H108, H107 to H109, H108 to H110, H109 to H111
Connections:
- H103 pad 1: unconnected-(H101-Pad1) -> Net-(H102-Pad1)
- H110 pad 1: unconnected-(H108-Pad1) -> Net-(J101-Pin_6)
Routing:
- net Net-(J101-Pin_6): track 0.00 -> 215.2 mm
- net Net-(J101-Pin_7): track 0.00 -> 160.4 mm
- net Net-(J101-Pin_5): track 0.00 -> 101.5 mm
- net Net-(J101-Pin_4): track 0.00 -> 78.6 mm
- net Net-(J101-Pin_3): track 0.00 -> 75.3 mm
- net Net-(J101-Pin_2): track 0.00 -> 56.0 mm
- net Net-(H102-Pad1): track 0.00 -> 25.4 mm
- net Net-(J101-Pin_1): track 0.00 -> 23.0 mm
- added copper zone on B.Cu, net (none)
- added copper zone on F.Cu, net (none)
Other:
- outline, holes or cut-outs redrawn

Commit message: rev2
Parts:
- moved H104 34.9 mm to (73.0, 34.9)
- moved H105 31.8 mm to (73.0, 69.8)
- moved H103 31.3 mm to (73.0, 104.8)
- moved J101 30.9 mm to (53.2, 40.6)
- moved H101 28.8 mm to (50.8, 72.8)
- moved H102 28.8 mm to (50.8, 102.8)
- moved H110 22.5 mm to (219.1, 34.9)
- moved H111 17.6 mm to (219.1, 69.8)
- moved H108 17.4 mm to (146.1, 34.9)
- moved H109 16.2 mm to (219.1, 104.8)
- moved G*** 13.7 mm to (188.0, 96.5)
- moved H107 8.98 mm to (146.1, 69.8)
- moved H106 7.10 mm to (146.1, 104.8)
Routing:
- net Net-(J101-Pin_7): track 160.4 -> 186.2 mm
- net Net-(J101-Pin_5): track 101.5 -> 126.2 mm
- net Net-(J101-Pin_4): track 78.6 -> 101.8 mm
- net Net-(J101-Pin_3): track 75.3 -> 97.2 mm
- net Net-(J101-Pin_6): track 215.2 -> 223.3 mm
- net Net-(H102-Pad1): track 25.4 -> 23.1 mm
- net Net-(J101-Pin_1): track 23.0 -> 22.1 mm
- net Net-(J101-Pin_2): track 56.0 -> 56.6 mm
- removed copper zone on B.Cu, net (none)
- removed copper zone on F.Cu, net (none)
Other:
- board size 152.4 x 76.2 mm -> 203.2 x 101.6 mm

Commit message: rev3
Parts:
- moved H109 72.0 mm to (147.0, 104.8)
- moved H110 72.0 mm to (147.0, 34.9)
- moved H111 72.0 mm to (147.0, 69.8)
- moved G*** 61.2 mm to (126.8, 94.7)
- moved H106 36.0 mm to (110.0, 104.8)
- moved H107 36.0 mm to (110.0, 69.8)
- moved H108 36.0 mm to (110.0, 34.9)
- moved H104 0.15 mm to (73.0, 34.8)
- moved H105 0.07 mm to (73.0, 69.8)
Routing:
- net Net-(J101-Pin_7): track 186.2 -> 146.6 mm
- net Net-(J101-Pin_4): track 101.8 -> 65.8 mm
- net Net-(J101-Pin_3): track 97.2 -> 61.2 mm
- net Net-(J101-Pin_5): track 126.2 -> 93.1 mm
- net Net-(J101-Pin_6): track 223.3 -> 201.6 mm
- net Net-(J101-Pin_2): track 56.6 -> 61.3 mm
- net Net-(J101-Pin_1): track 22.1 -> 24.0 mm
Other:
- board size 203.2 x 101.6 mm -> 130 x 100 mm
Changed lines of the file:
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@@
 		(pad_to_mask_clearance 0)
 		(allow_soldermask_bridges_in_footprints no)
+		(grid_origin 31.75 19.05)
 		(pcbplotparams
 			(layerselection 0x00010fc_ffffffff)
@@
 	(footprint "MountingHole:MountingHole_6.4mm_M6_Pad_Via"
 		(layer "F.Cu")
-		(at 73.025 34.925)
+		(at 73.025 34.775)
 		(descr "Mounting Hole 6.4mm, M6")
 		(tags "mounting hole 6.4mm m6")
@@
 	(footprint "MountingHole:MountingHole_4.3mm_M4_Pad_Via"
 		(layer "F.Cu")
-		(at 146.05 34.925)
+		(at 110.025 34.925)
 		(descr "Mounting Hole 4.3mm, M4")
 		(tags "mounting hole 4.3mm m4")
@@
 	(footprint "Symbol:prs_logo_shitty"
 		(layer "F.Cu")
-		(at 187.96 96.52)
+		(at 126.808459 94.686378)
 		(property "Reference" "G***"
 			(at 0 0 0)
@@
 	(footprint "MountingHole:MountingHole_6.4mm_M6_Pad_Via"
 		(layer "F.Cu")
-		(at 219.075 34.925)
+		(at 147.025 34.925)
 		(descr "Mounting Hole 6.4mm, M6")
 		(tags "mounting hole 6.4mm m6")
@@
 	(footprint "MountingHole:MountingHole_6.4mm_M6_Pad_Via"
 		(layer "F.Cu")
-		(at 219.075 104.775)
+		(at 147.025 104.775)
 		(descr "Mounting Hole 6.4mm, M6")
 		(tags "mounting hole 6.4mm m6")
@@
 	(footprint "MountingHole:MountingHole_4.3mm_M4_Pad_Via"
 		(layer "F.Cu")
-		(at 146.05 104.775)
+		(at 110.025 104.775)
 		(descr "Mounting Hole 4.3mm, M4")
 		(tags "mounting hole 4.3mm m4")
@@
 	(footprint "MountingHole:MountingHole_6.4mm_M6_Pad_Via"
 		(layer "F.Cu")
-		(at 73.025 69.85)
+		(at 73.025 69.775)
 		(descr "Mounting Hole 6.4mm, M6")
 		(tags "mounting hole 6.4mm m6")
@@
 	(footprint "MountingHole:MountingHole_4.3mm_M4_Pad_Via"
 		(layer "F.Cu")
-		(at 146.05 69.85)
+		(at 110.025 69.85)
 		(descr "Mounting Hole 4.3mm, M4")
 		(tags "mounting hole 4.3mm m4")
@@
 	(footprint "MountingHole:MountingHole_6.4mm_M6_Pad_Via"
 		(layer "F.Cu")
-		(at 219.075 69.85)
+		(at 147.025 69.85)
 		(descr "Mounting Hole 6.4mm, M6")
 		(tags "mounting hole 6.4mm m6")
@@
 	)
 	(gr_line
-		(start 31.75 19.05)
-		(end 234.95 19.05)
+		(start 31.75 21.55)
+		(end 161.75 21.55)
 		(stroke
 			(width 0.1)
@@
 	)
 	(gr_line
-		(start 234.95 19.05)
-		(end 234.95 120.65)
+		(start 161.75 21.55)
+		(end 161.75 121.55)
 		(stroke
 			(width 0.1)
@@
 	)
 	(gr_line
-		(start 31.75 120.65)
-		(end 31.75 19.05)
+		(start 31.75 121.55)
+		(end 31.75 21.55)
 		(stroke
 			(width 0.1)
@@
 	)
 	(gr_line
-		(start 234.95 120.65)
-		(end 31.75 120.65)
+		(start 161.75 121.55)
+		(end 31.75 121.55)
 		(stroke
 			(width 0.1)
@@
 	)
 	(gr_text "PRS Leaf Battery Thing"
-		(at 157.48 86.36 0)
+		(at 96.328459 84.526378 0)
 		(layer "F.SilkS")
 		(effects
@@
 	)
 	(segment
-		(start 67.31 40.64)
-		(end 73.025 34.925)
-		(width 0.508)
+		(start 56 34.775)
+		(end 73.025 34.775)
+		(width 1)
+		(layer "F.Cu")
+		(net 2)
+	)
+	(segment
+		(start 53.25 37.525)
+		(end 56 34.775)
+		(width 1)
 		(layer "F.Cu")
 		(net 2)
@@
 	(segment
 		(start 53.25 40.64)
-		(end 67.31 40.64)
-		(width 0.508)
+		(end 53.25 37.525)
+		(width 1)
 		(layer "F.Cu")
 		(net 2)
 	)
 	(segment
-		(start 70.125 72.75)
-		(end 73.025 69.85)
+		(start 50.78 72.75)
+		(end 70.05 72.75)
 		(width 13)
 		(layer "F.Cu")
@@
 	)
 	(segment
-		(start 50.78 63.25)
-		(end 50.78 72.75)
-		(width 0.508)
+		(start 70.05 72.75)
+		(end 73.025 69.775)
+		(width 13)
 		(layer "F.Cu")
 		(net 3)
@@
 	(segment
 		(start 53.25 43.14)
-		(end 47.71 48.68)
-		(width 0.508)
+		(end 51.285 43.14)
+		(width 1)
 		(layer "F.Cu")
 		(net 3)
 	)
 	(segment
-		(start 50.78 72.75)
-		(end 70.125 72.75)
-		(width 13)
+		(start 51.285 43.14)
+		(end 43.475 50.95)
+		(width 1)
 		(layer "F.Cu")
 		(net 3)
 	)
 	(segment
-		(start 47.71 48.68)
-		(end 47.71 60.18)
-		(width 0.508)
+		(start 43.475 65.445)
+		(end 50.78 72.75)
+		(width 1)
 		(layer "F.Cu")
 		(net 3)
 	)
 	(segment
-		(start 47.71 60.18)
-		(end 50.78 63.25)
-		(width 0.508)
+		(start 43.475 50.95)
+		(end 43.475 65.445)
+		(width 1)
 		(layer "F.Cu")
 		(net 3)
@@
 	(segment
 		(start 53.25 50.64)
-		(end 50.5 50.64)
-		(width 0.508)
+		(end 79.54 50.64)
+		(width 1)
 		(layer "F.Cu")
 		(net 4)
 	)
 	(segment
-		(start 131.855 104.775)
-		(end 146.05 104.775)
-		(width 0.508)
+		(start 110.025 81.125)
+		(end 110.025 104.775)
+		(width 1)
 		(layer "F.Cu")
 		(net 4)
 	)
 	(segment
-		(start 50.5 50.64)
-		(end 49.6 51.54)
-		(width 0.508)
+		(start 79.54 50.64)
+		(end 110.025 81.125)
+		(width 1)
 		(layer "F.Cu")
 		(net 4)
 	)
 	(segment
-		(start 49.6 57.78)
-		(end 51.42 59.6)
-		(width 0.508)
+		(start 88.315 48.14)
+		(end 110.025 69.85)
+		(width 1)
 		(layer "F.Cu")
-		(net 4)
+		(net 5)
 	)
 	(segment
-		(start 86.68 59.6)
-		(end 131.855 104.775)
-		(width 0.508)
+		(start 53.25 48.14)
+		(end 88.315 48.14)
+		(width 1)
 		(layer "F.Cu")
-		(net 4)
+		(net 5)
 	)
 	(segment
-		(start 49.6 51.54)
-		(end 49.6 57.78)
-		(width 0.508)
+		(start 53.25 45.64)
+		(end 99.31 45.64)
+		(width 1)
 		(layer "F.Cu")
-		(net 4)
+		(net 6)
 	)
 	(segment
-		(start 51.42 59.6)
-		(end 86.68 59.6)
-		(width 0.508)
+		(start 99.31 45.64)
+		(end 110.025 34.925)
+		(width 1)
 		(layer "F.Cu")
-		(net 4)
+		(net 6)
 	)
 	(segment
-		(start 124.34 48.14)
-		(end 146.05 69.85)
-		(width 0.508)
+		(start 97.8 117.475)
+		(end 128.75 117.475)
+		(width 1)
 		(layer "F.Cu")
-		(net 5)
+		(net 7)
 	)
 	(segment
-		(start 53.25 48.14)
-		(end 124.34 48.14)
-		(width 0.508)
+		(start 87.25 106.925)
+		(end 97.8 117.475)
+		(width 1)
 		(layer "F.Cu")
-		(net 5)
+		(net 7)
 	)
 	(segment
-		(start 111.14 45.64)
-		(end 121.855 34.925)
-		(width 0.508)
+		(start 87.25 69.4)
+		(end 87.25 106.925)
+		(width 1)
 		(layer "F.Cu")
-		(net 6)
+		(net 7)
 	)
 	(segment
-		(start 121.855 34.925)
-		(end 146.05 34.925)
-		(width 0.508)
+		(start 53.25 55.64)
+		(end 73.49 55.64)
+		(width 1)
 		(layer "F.Cu")
-		(net 6)
+		(net 7)
 	)
 	(segment
-		(start 53.25 45.64)
-		(end 111.14 45.64)
-		(width 0.508)
+		(start 138.25 113.55)
+		(end 147.025 104.775)
+		(width 1)
 		(layer "F.Cu")
-		(net 6)
+		(net 7)
 	)
 	(segment
-		(start 156.42 91.32)
-		(end 169.875 104.775)
-		(width 0.508)
+		(start 132.675 113.55)
+		(end 138.25 113.55)
+		(width 1)
 		(layer "F.Cu")
 		(net 7)
 	)
 	(segment
-		(start 88.33 55.64)
-		(end 124.01 91.32)
-		(width 0.508)
+		(start 128.75 117.475)
+		(end 132.675 113.55)
+		(width 1)
 		(layer "F.Cu")
 		(net 7)
 	)
 	(segment
-		(start 169.875 104.775)
-		(end 219.075 104.775)
-		(width 0.508)
+		(start 73.49 55.64)
+		(end 87.25 69.4)
+		(width 1)
 		(layer "F.Cu")
 		(net 7)
 	)
 	(segment
-		(start 53.25 55.64)
-		(end 88.33 55.64)
-		(width 0.508)
+		(start 122.3 113.05)
+		(end 147.025 88.325)
+		(width 1)
 		(layer "F.Cu")
-		(net 7)
+		(net 8)
 	)
 	(segment
-		(start 124.01 91.32)
-		(end 156.42 91.32)
-		(width 0.508)
+		(start 53.25 53.14)
+		(end 75.615 53.14)
+		(width 1)
 		(layer "F.Cu")
-		(net 7)
+		(net 8)
 	)
 	(segment
-		(start 53.25 53.14)
-		(end 88.4 53.14)
-		(width 0.508)
+		(start 102.4 113.05)
+		(end 122.3 113.05)
+		(width 1)
 		(layer "F.Cu")
 		(net 8)
 	)
 	(segment
-		(start 219.075 34.925)
-		(end 219.075 69.85)
-		(width 13)
+		(start 92.55 70.075)
+		(end 92.55 103.2)
+		(width 1)
 		(layer "F.Cu")
 		(net 8)
 	)
 	(segment
-		(start 124.01 88.75)
-		(end 165.13 88.75)
-		(width 0.508)
+		(start 75.615 53.14)
+		(end 92.55 70.075)
+		(width 1)
 		(layer "F.Cu")
 		(net 8)
 	)
 	(segment
-		(start 88.4 53.14)
-		(end 124.01 88.75)
-		(width 0.508)
+		(start 147.025 88.325)
+		(end 147.025 69.85)
+		(width 1)
 		(layer "F.Cu")
 		(net 8)
 	)
 	(segment
-		(start 184.03 69.85)
-		(end 219.075 69.85)
-		(width 0.508)
+		(start 147.025 69.85)
+		(end 147.025 34.925)
+		(width 13)
 		(layer "F.Cu")
 		(net 8)
 	)
 	(segment
-		(start 165.13 88.75)
-		(end 184.03 69.85)
-		(width 0.508)
+		(start 92.55 103.2)
+		(end 102.4 113.05)
+		(width 1)
 		(layer "F.Cu")
 		(net 8)
